File: projects/wanos-board/water_meters.kicad_sch (KiCad schematic)
At the start: 20 parts

Commit message: add RJ45 & TVS
Parts:
- added D25, D26, D27, D28: PESD5V0S1BA, Diode_SMD:D_SOD-323, symbol Device:D_TVS
- added D29: SMBJ5.0A, Diode_SMD:D_SMB, symbol Device:D_TVS
- added J4: WATER_RJ45, Connector_RJ:RJ45_Amphenol_RJHSE5380, symbol Connector_Generic:Conn_01x08
Connections:
- net +3V3: no longer R19.1, R20.1, R21.1, R22.1, R37.1, R38.1, R39.1, R40.1
- net EXP_A_P2_WM_B1_COLD: no longer R37.2, R41.2, R42.1
- net EXP_A_P3_WM_B1_HOT: no longer R38.2, R42.2, R43.1
- net EXP_A_P4_WM_B2_COLD: no longer R39.2, R43.2, R44.1
- net EXP_A_P5_WM_B2_HOT: no longer R40.2, R44.2
- net WM_B1_COLD: no longer R41.1
Other:
- note added: "B1 COLD"
- note added: "B1 HOT"
- note added: "B2 COLD"
- note added: "B2 HOT"
- note added: "Cat5 ~10m; YF OD + 3V3 pull-up; TVS D25-D28 SIG, D29 +5VA; no MOSFET"
- note added: "D29 +5VA clamp"
- note added: "J4 RJ45 (T568B): 1=B1_COLD 2=GND 3=B1_HOT 4=+5VA 5=GND 6=GND 7=B2_COLD 8=B2_HOT; SH->GND"
- note removed: "B1 COLD / J4"
- note removed: "B1 HOT / J4"
- note removed: "B2 COLD / J5"
- note removed: "B2 HOT / J5"
- note removed: "Field nets WM_* leave connectors J4/J5; EXP_A_P* enter U1 on IO_Expanders"
- note removed: "J4/J5 pinout: 1=GND 2=COLD SIG 3=HOT SIG 4=+5VA 5=GND 6=+5VA (connectors sheet)"
- note removed: "Sensor VDD = +5VA on J4/J5 (not on this netlist node — harness)"
- note removed: "YF-B6/B10 — OD to +3V3 pull-up, 330 series, 100n debounce, LED (no MOSFET)"

Commit message: watermeters schematic 2nd pass
Parts:
- J4: value WATER_RJ45 -> 5556416-1; footprint Connector_RJ:RJ45_Amphenol_RJHSE5380 -> Connector_RJ:RJ45_Amphenol_54602-x08_Horizontal
Connections:
- net +3V3: now also R19.1, R20.1, R21.1, R22.1, R37.1, R38.1, R39.1, R40.1
- net +5VA: now also D29.1 (A1), J4.4 (Pin_4)
- net EXP_A_P2_WM_B1_COLD: now also D13.2 (A), R41.2
- net EXP_A_P3_WM_B1_HOT: now also D14.2 (A), R42.2
- net EXP_A_P4_WM_B2_COLD: now also D15.2 (A), R43.2
- net EXP_A_P5_WM_B2_HOT: now also D16.2 (A), R44.2
- net GND: now also C18.2, C19.2, C20.2, C21.2, D25.2 (A2), D26.2 (A2), D27.2 (A2), D28.2 (A2), D29.2 (A2), J4.2 (Pin_2), J4.5 (Pin_5), J4.6 (Pin_6)
- net WM_B1_COLD: now also C18.1, D25.1 (A1), J4.1 (Pin_1), R37.2, R41.1
- net WM_B1_HOT: now also C19.1, D26.1 (A1), J4.3 (Pin_3), R38.2, R42.1
- net WM_B2_COLD: now also C20.1, D27.1 (A1), J4.7 (Pin_7), R39.2, R43.1
- net WM_B2_HOT: now also C21.1, D28.1 (A1), J4.8 (Pin_8), R40.2, R44.1
- new net: D16.1 (K), R22.2
- new net: D14.1 (K), R20.2
- new net: D13.1 (K), R19.2
- new net: D15.1 (K), R21.2
Other:
- note added: "J4 TE 5556416-1 (LCSC C86492) TH RJ45 no LED; fp RJ45_Amphenol_54602-x08_Horizontal"
- note added: "T568B: 1=B1_COLD 2=GND 3=B1_HOT 4=+5VA 5=GND 6=GND 7=B2_COLD 8=B2_HOT"
- note removed: "Cat5 ~10m; YF OD + 3V3 pull-up; TVS D25-D28 SIG, D29 +5VA; no MOSFET"
- note removed: "D29 +5VA clamp"
- note removed: "J4 RJ45 (T568B): 1=B1_COLD 2=GND 3=B1_HOT 4=+5VA 5=GND 6=GND 7=B2_COLD 8=B2_HOT; SH->GND"

Commit message: adjusted water schema add datasheets
Other:
- note removed: "J4 TE 5556416-1 (LCSC C86492) TH RJ45 no LED; fp RJ45_Amphenol_54602-x08_Horizontal"
- note removed: "T568B: 1=B1_COLD 2=GND 3=B1_HOT 4=+5VA 5=GND 6=GND 7=B2_COLD 8=B2_HOT"
- moved on the sheet: C18, C19, C20, C21, D13, D14, D15, D16, D25, D26, D27, D28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
