File: projects/wanos-board/wanos-board.kicad_sch (KiCad schematic)
At the start: 0 parts

Commit message: SSR, power, IO_expander schemas update
Other:
- removed sheet LEDs
- removed sheet Safety_12V_Mon
Changed lines of the file:
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@@
-	)
-	(sheet
-		(at 235 75)
-		(size 60 40)
-		(exclude_from_sim no)
-		(in_bom yes)
-		(on_board yes)
-		(dnp no)
-		(fields_autoplaced yes)
-		(stroke
-			(width 0.1524)
-			(type solid)
-		)
-		(fill
-			(color 0 0 0 0)
-		)
-		(property "Sheetname" "LEDs"
-			(at 235 74.365 0)
-			(show_name no)
-			(do_not_autoplace no)
-			(effects
-				(font
-					(size 1.27 1.27)
-				)
-				(justify left bottom)
-			)
-		)
-		(property "Sheetfile" "leds.kicad_sch"
-			(at 235 115.635 0)
-			(show_name no)
-			(do_not_autoplace no)
-			(effects
-				(font
-					(size 1.27 1.27)
-				)
-				(justify left top)
-			)
-		)
-		(instances
-			(project "wanos-board"
-				(path "/b64fe9be-4bba-4a4c-aa66-7fa6f4bbb662"
-					(page "9")
-				)
-			)
-		)
 	)
 	(sheet
@@
 				)
 			)
-		)
-	)
-	(sheet
-		(at 235 25)
-		(size 60 40)
-		(exclude_from_sim no)
-		(in_bom yes)
-		(on_board yes)
-		(dnp no)
-		(fields_autoplaced yes)
-		(stroke
-			(width 0.1524)
-			(type solid)
-		)
-		(fill
-			(color 0 0 0 0)
-		)
-		(property "Sheetname" "Safety_12V_Mon"
-			(at 235 24.365 0)
-			(show_name no)
-			(do_not_autoplace no)
-			(effects
-				(font
-					(size 1.27 1.27)
-				)
-				(justify left bottom)
-			)
-		)
-		(property "Sheetfile" "safety_12v_mon.kicad_sch"
-			(at 235 65.635 0)
-			(show_name no)
-			(do_not_autoplace no)
-			(effects
-				(font
-					(size 1.27 1.27)
-				)
-				(justify left top)
-			)
-		)
-		(instances
-			(project "wanos-board"
-				(path "/b64fe9be-4bba-4a4c-aa66-7fa6f4bbb662"
-					(page "6")
-				)
-			)

Commit message: 1st draft: water meters schematic
Other:
- added sheet Water_Meters (water_meters.kicad_sch)
Changed lines of the file:
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@@
+		)
+	)
+	(sheet
+		(at 235 25)
+		(size 60 40)
+		(exclude_from_sim no)
+		(in_bom yes)
+		(on_board yes)
+		(dnp no)
+		(fields_autoplaced yes)
+		(stroke
+			(width 0.1524)
+			(type solid)
+		)
+		(fill
+			(color 0 0 0 0)
+		)
+		(property "Sheetname" "Water_Meters"
+			(at 235 24.365 0)
+			(show_name no)
+			(do_not_autoplace no)
+			(effects
+				(font
+					(size 1.27 1.27)
+				)
+				(justify left bottom)
+			)
+		)
+		(property "Sheetfile" "water_meters.kicad_sch"
+			(at 235 65.635 0)
+			(show_name no)
+			(do_not_autoplace no)
+			(effects
+				(font
+					(size 1.27 1.27)
+				)
+				(justify left top)
+			)
+		)
+		(instances
+			(project "wanos-board"
+				(path "/b64fe9be-4bba-4a4c-aa66-7fa6f4bbb662"
+					(page "6")
+				)
+			)
 		)
 	)

Commit message: schema updates
Other:
- sheet Water_Meters renamed Pulse_Inputs
- removed sheet Connectors
- sheet Pulse_Inputs: file water_meters.kicad_sch -> pulse_inputs.kicad_sch
Changed lines of the file:
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@@
-	)
-	(sheet
-		(at 165 75)
-		(size 60 40)
-		(exclude_from_sim no)
-		(in_bom yes)
-		(on_board yes)
-		(dnp no)
-		(fields_autoplaced yes)
-		(stroke
-			(width 0.1524)
-			(type solid)
-		)
-		(fill
-			(color 0 0 0 0)
-		)
-		(property "Sheetname" "Connectors"
-			(at 165 74.365 0)
-			(show_name no)
-			(do_not_autoplace no)
-			(effects
-				(font
-					(size 1.27 1.27)
-				)
-				(justify left bottom)
-			)
-		)
-		(property "Sheetfile" "connectors.kicad_sch"
-			(at 165 115.635 0)
-			(show_name no)
-			(do_not_autoplace no)
-			(effects
-				(font
-					(size 1.27 1.27)
-				)
-				(justify left top)
-			)
-		)
-		(instances
-			(project "wanos-board"
-				(path "/b64fe9be-4bba-4a4c-aa66-7fa6f4bbb662"
-					(page "8")
-				)
-			)
-		)
 	)
 	(sheet
@@
 			(color 0 0 0 0)
 		)
-		(property "Sheetname" "Water_Meters"
+		(property "Sheetname" "Pulse_Inputs"
 			(at 235 24.365 0)
 			(show_name no)
@@
 			)
 		)
-		(property "Sheetfile" "water_meters.kicad_sch"
+		(property "Sheetfile" "pulse_inputs.kicad_sch"
 			(at 235 65.635 0)
 			(show_name no)
